Commit message: new code for new mc

File: src/urdf/robot.urdf (robot description, URDF)
Before this commit: robot robot, 4 links, 3 joints
Links:
- removed link back_wheel
- removed link left_wheel
- removed link right_wheel
Joints:
- removed joint back_wheel_join
- removed joint left_wheel_joint
- removed joint right_wheel_joint
